File: HV2907_preamp/HV2907_preamp.kicad_sch (KiCad schematic)
At the start: 48 parts, among them J1 Mic Input, J2 HI-Z Input, J3 Output, Q1 BC548, Q2 BF246A, Q3 2SA1015, SW1 Phantom Power, SW2 -20dB PAD, SW3 Boost, T1 Jensen JT-115K-EPC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

Commit message: HV2907 circuit update
Parts:
- removed SW3: Boost, symbol Switch:SW_SPDT
- added RV2: 250KB, symbol Device:R_Potentiometer
- R10: value 10K -> 20K
- R11: value 10K -> 47K
- RV1: value Level -> 100KB
Connections:
- net GND: now also RV2.2, RV2.3
- net at C7.2, R11.2: now also RV2.1
Other:
- note added: "Level"
- note added: "Tube Gain"
Changed lines of the file:
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@@
 	(generator_version "9.0")
 	(paper "A4")
+	(text "Tube Gain"
+		(exclude_from_sim no)
+		(at 183.388 141.478 0)
+		(effects
+			(font
+				(size 1.27 1.27)
+			)
+		)
+	)
+	(text "Level"
+		(exclude_from_sim no)
+		(at 198.374 124.46 0)
+		(effects
+			(font
+				(size 1.27 1.27)
+			)
+		)
+	)
 	(junction
 		(at 173.99 72.39)
@@
 	)
 	(junction
-		(at 177.8 148.59)
+		(at 158.75 148.59)
 		(diameter 0)
 		(color 0 0 0 0)
 	)
 	(junction
-		(at 158.75 148.59)
+		(at 110.49 134.62)
 		(diameter 0)
 		(color 0 0 0 0)
 	)
 	(junction
-		(at 167.64 134.62)
+		(at 147.32 111.76)
 		(diameter 0)
 		(color 0 0 0 0)
 	)
 	(junction
-		(at 110.49 134.62)
+		(at 88.9 114.3)
 		(diameter 0)
 		(color 0 0 0 0)
 	)
 	(junction
-		(at 147.32 111.76)
+		(at 238.76 123.19)
 		(diameter 0)
 		(color 0 0 0 0)
 	)
 	(junction
-		(at 88.9 114.3)
+		(at 173.99 148.59)
 		(diameter 0)
 		(color 0 0 0 0)
 	)
 	(junction
-		(at 238.76 123.19)
+		(at 81.28 101.6)
 		(diameter 0)
 		(color 0 0 0 0)
 	)
 	(junction
-		(at 81.28 101.6)
+		(at 167.64 134.62)
 		(diameter 0)
 		(color 0 0 0 0)
@@
 	)
 	(junction
+		(at 177.8 148.59)
+		(diameter 0)
+		(color 0 0 0 0)
+	)
+	(junction
 		(at 39.37 46.99)
 		(diameter 0)
@@
 	(wire
 		(pts
+			(xy 173.99 134.62) (xy 167.64 134.62)
+		)
+		(stroke
+			(width 0)
+			(type default)
+		)
+	)
+	(wire
+		(pts
 			(xy 218.44 137.16) (xy 224.79 137.16)
 		)
@@
 	(wire
 		(pts
+			(xy 177.8 139.7) (xy 177.8 148.59)
+		)
+		(stroke
+			(width 0)
+			(type default)
+		)
+	)
+	(wire
+		(pts
 			(xy 266.7 140.97) (xy 266.7 151.13)
 		)
@@
 	(wire
 		(pts
-			(xy 177.8 144.78) (xy 177.8 148.59)
+			(xy 173.99 60.96) (xy 173.99 59.69)
 		)
 		(stroke
@@
 	(wire
 		(pts
-			(xy 173.99 60.96) (xy 173.99 59.69)
+			(xy 146.05 148.59) (xy 146.05 149.86)
 		)
 		(stroke
@@
 	(wire
 		(pts
-			(xy 146.05 148.59) (xy 146.05 149.86)
+			(xy 53.34 39.37) (xy 55.88 39.37)
 		)
 		(stroke
@@
 	(wire
 		(pts
-			(xy 53.34 39.37) (xy 55.88 39.37)
+			(xy 248.92 148.59) (xy 218.44 148.59)
 		)
 		(stroke
@@
 	(wire
 		(pts
-			(xy 248.92 148.59) (xy 218.44 148.59)
+			(xy 85.09 137.16) (xy 85.09 149.86)
 		)
 		(stroke
@@
 	(wire
 		(pts
-			(xy 85.09 137.16) (xy 85.09 149.86)
+			(xy 154.94 78.74) (xy 154.94 101.6)
 		)
 		(stroke
@@
 	(wire
 		(pts
-			(xy 154.94 78.74) (xy 154.94 101.6)
+			(xy 177.8 148.59) (xy 186.69 148.59)
 		)
 		(stroke
@@
 	(wire
 		(pts
+			(xy 173.99 148.59) (xy 177.8 148.59)
+		)
+		(stroke
+			(width 0)
+			(type default)
+		)
+	)
+	(wire
+		(pts
 			(xy 173.99 72.39) (xy 173.99 76.2)
 		)
@@
 	(wire
 		(pts
-			(xy 167.64 134.62) (xy 167.64 135.89)
-		)
-		(stroke
-			(width 0)
-			(type default)
-		)
-	)
-	(wire
-		(pts
 			(xy 147.32 111.76) (xy 147.32 88.9)
 		)
@@
 	(wire
 		(pts
-			(xy 167.64 134.62) (xy 180.34 134.62)
+			(xy 73.66 74.93) (xy 73.66 72.39)
 		)
 		(stroke
@@
 	(wire
 		(pts
-			(xy 73.66 74.93) (xy 73.66 72.39)
+			(xy 152.4 125.73) (xy 152.4 111.76)
 		)
 		(stroke
@@
 	(wire
 		(pts
-			(xy 152.4 125.73) (xy 152.4 111.76)
+			(xy 86.36 114.3) (xy 88.9 114.3)
 		)
 		(stroke
@@
 	(wire
 		(pts
-			(xy 86.36 114.3) (xy 88.9 114.3)
+			(xy 167.64 134.62) (xy 167.64 135.89)
 		)
 		(stroke
@@
 	(wire
 		(pts
+			(xy 173.99 143.51) (xy 173.99 148.59)
+		)
+		(stroke
+			(width 0)
+			(type default)
+		)
+	)
+	(wire
+		(pts
 			(xy 34.29 121.92) (xy 90.17 121.92)
 		)
@@
 	(wire
 		(pts
-			(xy 72.39 110.49) (xy 72.39 114.3)
+			(xy 173.99 135.89) (xy 173.99 134.62)
 		)
 		(stroke
@@
 	(wire
 		(pts
-			(xy 147.32 114.3) (xy 147.32 111.76)
+			(xy 72.39 110.49) (xy 72.39 114.3)
 		)
 		(stroke
@@
 	(wire
 		(pts
-			(xy 88.9 114.3) (xy 90.17 114.3)
+			(xy 147.32 114.3) (xy 147.32 111.76)
 		)
 		(stroke
@@
 	(wire
 		(pts
-			(xy 46.99 101.6) (xy 46.99 102.87)
+			(xy 88.9 114.3) (xy 90.17 114.3)
 		)
 		(stroke
@@
 	(wire
 		(pts
-			(xy 186.69 148.59) (xy 177.8 148.59)
+			(xy 46.99 101.6) (xy 46.99 102.87)
 		)
 		(stroke
@@
 	(wire
 		(pts
-			(xy 34.29 111.76) (xy 34.29 121.92)
+			(xy 167.64 148.59) (xy 173.99 148.59)
 		)
 		(stroke
@@
 	(wire
 		(pts
-			(xy 63.5 58.42) (xy 63.5 53.34)
+			(xy 34.29 111.76) (xy 34.29 121.92)
 		)
 		(stroke
@@
 	(wire
 		(pts
-			(xy 114.3 116.84) (xy 110.49 116.84)
+			(xy 63.5 58.42) (xy 63.5 53.34)
 		)
 		(stroke
@@
 	(wire
 		(pts
-			(xy 154.94 68.58) (xy 154.94 71.12)
+			(xy 114.3 116.84) (xy 110.49 116.84)
 		)
 		(stroke
@@
 	(wire
 		(pts
-			(xy 177.8 148.59) (xy 167.64 148.59)
+			(xy 154.94 68.58) (xy 154.94 71.12)
 		)
 		(stroke
@@
 			)
 		)
-		(property "Value" "Level"
+		(property "Value" "100KB"
 			(at 201.422 121.666 0)
 			(effects
@@
 			)
 		)
-		(property "Value" "10K"
+		(property "Value" "47K"
 			(at 162.306 140.97 0)
 			(effects
@@
 			)
 		)
-		(property "Value" "10K"
+		(property "Value" "20K"
 			(at 152.908 140.97 0)
 			(effects
@@
 	)
 	(symbol
+		(lib_id "Device:R_Potentiometer")
+		(at 173.99 139.7 0)
+		(unit 1)
+		(exclude_from_sim no)
+		(in_bom yes)
+		(on_board yes)
+		(dnp no)
+		(property "Reference" "RV2"
+			(at 180.594 134.112 0)
+			(effects
+				(font
+					(size 1.27 1.27)
+				)
+				(justify right)
+			)
+		)
+		(property "Value" "250KB"
+			(at 183.134 136.398 0)
+			(effects
+				(font
+					(size 1.27 1.27)
+				)
+				(justify right)
+			)
+		)
+		(property "Footprint" ""
+			(at 173.99 139.7 0)
+			(effects
+				(font
+					(size 1.27 1.27)
+				)
+				(hide yes)
+			)
+		)
+		(property "Datasheet" "~"
+			(at 173.99 139.7 0)
+			(effects
+				(font
+					(size 1.27 1.27)
+				)
+				(hide yes)
+			)
+		)
+		(property "Description" "Potentiometer"
+			(at 173.99 139.7 0)
+			(effects
+				(font
+					(size 1.27 1.27)
+				)
+				(hide yes)
+			)
+		)
+		(pin "3"
+		)
+		(pin "2"
+		)
+		(pin "1"
+		)
+		(instances
+			(project ""
+				(path "/ba57b884-0e6b-4b46-b520-20662842143e"
+					(reference "RV2")
+					(unit 1)
+				)
+			)
+		)
+	)
+	(symbol
 		(lib_id "Device:R")
 		(at 186.69 120.65 180)
@@
 					(unit 1)
 				)
-			)
-		)
-	)
-	(symbol
-		(lib_id "Switch:SW_SPDT")
-		(at 180.34 139.7 270)
-		(unit 1)
-		(exclude_from_sim no)
-		(in_bom yes)
-		(on_board yes)
-		(dnp no)
-		(property "Reference" "SW3"
-			(at 185.166 139.7 90)
-			(effects
-				(font
-					(size 1.27 1.27)
-				)
-				(justify left)
-			)
-		)
-		(property "Value" "Boost"
-			(at 184.912 141.986 90)
-			(effects
-				(font
-					(size 1.27 1.27)
-				)
-				(justify left)
-			)
-		)
-		(property "Footprint" ""
-			(at 180.34 139.7 0)
-			(effects
-				(font
-					(size 1.27 1.27)
-				)
-				(hide yes)
-			)
-		)
-		(property "Datasheet" "~"
-			(at 172.72 139.7 0)
-			(effects
-				(font
-					(size 1.27 1.27)
-				)
-				(hide yes)
-			)
-		)
-		(property "Description" "Switch, single pole double throw"
-			(at 180.34 139.7 0)
-			(effects
-				(font
-					(size 1.27 1.27)
-				)
-				(hide yes)
-			)
-		)
-		(pin "3"
-		)
-		(pin "2"
-		)
-		(pin "1"
-		)
-		(instances
-			(project "HV2907_preamp"
-				(path "/ba57b884-0e6b-4b46-b520-20662842143e"
-					(reference "SW3")
-					(unit 1)
-				)

Commit message: New modifications to HV2907 preamp
Parts:
- added C13: 47uF X 35V, symbol Device:C_Polarized
- C12: value 4,7nF -> 470pF
- C7: value 100uF X 25V -> 47uF X 35V
- R13: value 50k -> 47K
- R16: value 1K -> 2K2
Connections:
- net GND: now also C13.2; no longer R16.1
- new net: C13.1, R16.1
Other:
- moved on the sheet: C10, C9, R16, R17, R18, U1A

Commit message: Preamp sch updated
Parts:
- removed C6: 47uF X 25V, symbol Device:C_Polarized
- removed F1: Fuse, symbol Device:Fuse
- removed R11: 47K, symbol Device:R
- removed R15: 10K, symbol Device:R
- added C14, C17, C20: 100uF X 35V, symbol Device:C_Polarized
- added C15, C18, C21: 1uF x 25V, symbol Device:C
- added C16, C19, C22: 100nF, symbol Device:C
- added D2, D3: 1N4007, Diode_THT:D_DO-41_SOD81_P10.16mm_Horizontal, symbol Diode:1N4007
- added Q4: TIP122, Package_TO_SOT_THT:TO-220-3_Vertical, symbol Transistor_BJT:TIP122
- added R22, R26: 100R, symbol Device:R
- added R23: 2.7K, symbol Device:R
- added R24: 1M, symbol Device:R
- added R25: 3.3K, symbol Device:R
- added unit 3 of U1
- added U2: L78L12_TO92, Package_TO_SOT_THT:TO-92_Inline, symbol Regulator_Linear:L78L12_TO92
- C11: value 4.7pF -> 47pF
- R17: value 10K -> 15K
- R18, R19, R20: value 150R -> 120R
- R5: value 1K -> 3K3
- RV1: value 100KB -> 10KA
- RV2: value 250KB -> 50KA
Connections:
- net +12V: now also V1.4, Q4.3 (E), R25.1
- net +15V: now also Q4.2 (C), R22.2, U2.3 (VI); no longer V1.6
- net GND: now also C14.1, C15.1, C16.1, C17.2, C18.1, C19.1, C20.1, C21.2, C22.2, D3.1 (K), R24.2, R25.2
- net at R12.1, V1.1: now also R23.2; no longer V1.7
- net at R14.2, R9.2, V1.2: now also T1.4 (SB)
- new net: R26.2, U2.1 (VO)
- new net: D2.2 (A), U2.2 (GND)
- new net: C20.2, C21.1, C22.1, U1.4 (V-)
- new net: C17.1, C18.2, C19.2, U1.8 (V+)
- new net: R23.1, R24.1, V1.7
- new net: D2.1 (K), D3.2 (A)
- new net: C14.2, C15.2, C16.2, R22.1, V1.6
- new net: Q4.1 (B), R26.1
Other:
- moved on the sheet: J3, R12, RV2, V1B
