File: channel_psu/channel_psu/channel_psu.kicad_sch (KiCad schematic)
At the start: 25 parts, among them J1 AC IN, J2 To DC-DC Step UP, J3 PSU Output, Q1 TIP42, Q2 TIP41, U1 LM7815_TO220, U2 L7915

Commit message: Preamp sch updated
Changed lines of the file:
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@@
 (kicad_sch
-	(version 20231120)
+	(version 20250114)
 	(generator "eeschema")
-	(generator_version "8.0")
+	(generator_version "9.0")
 	(paper "A4")
+	(text "+48V\n+15VDC\nGND\n-15VDC\n"
+		(exclude_from_sim no)
+		(at 211.582 95.504 0)
+		(effects
+			(font
+				(size 1.524 1.524)
+			)
+			(justify left)
+		)
+	)
+	(text "+V\nGND\nGND\n48VDC"
+		(exclude_from_sim no)
+		(at 211.328 57.15 0)
+		(effects
+			(font
+				(size 1.524 1.524)
+			)
+			(justify left)
+		)
+	)
 	(junction
 		(at 114.3 78.74)
@@
 		)
 	)
-	(text "+48V\n+15VDC\nGND\n-15VDC\n"
-		(exclude_from_sim no)
-		(at 211.582 95.504 0)
-		(effects
-			(font
-				(size 1.524 1.524)
-			)
-			(justify left)
-		)
-	)
-	(text "+V\nGND\nGND\n48VDC"
-		(exclude_from_sim no)
-		(at 211.328 57.15 0)
-		(effects
-			(font
-				(size 1.524 1.524)
-			)
-			(justify left)
-		)
-	)
 	(symbol
 		(lib_id "Device:C_Polarized")
@@
 		)
 	)
+	(embedded_fonts no)
 )
